File: minidexed.kicad_pcb (KiCad board)
At the start: 2 copper layers, 130.8 x 81.5 mm, 53 parts, among them J1 Audio Out, J2 MIDI In, J3 Raspberry_Pi_2_3, J4 MIDI Thru, J5 MIDI Out, J6 GND TP, SW1 Encoder, SW2 B1, SW3 B2, SW4 B3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

Commit message: jacks jlc
Parts:
- J1, J2, J4, J5: footprint sparkfun 3.5mm:sparkfun_3.5mm_trs -> jlcjack:PJ-320A
- moved J5 8.88 mm to (140.0, 66.2), turned to -90 degrees
- moved J1 6.81 mm to (155.5, 66.2), turned to -90 degrees
- moved J4 5.54 mm to (122.5, 66.2), turned to -90 degrees
- moved J2 4.19 mm to (107.0, 66.2), turned to -90 degrees
- moved R4 1.96 mm to (153.0, 75.0), turned to 180 degrees
- moved C14 1.45 mm to (158.9, 74.5)
- moved R6 1.29 mm to (103.5, 74.0)
- moved R11 1.12 mm to (136.0, 74.0)
- moved R10 1.11 mm to (123.0, 74.0), turned to 0 degrees
- moved R13 0.45 mm to (117.0, 73.5)
- moved D1 0.45 mm to (110.7, 73.5)
Routing:
- net Net-(J5-Pad2): track 4.49 -> 12.0 mm
- net Net-(C15-Pad1): track 9.40 -> 15.1 mm
- net Net-(J2-Pad2): track 4.57 -> 9.15 mm
- net Net-(J4-Pad2): track 3.95 -> 8.23 mm
- net Net-(C14-Pad1): track 9.64 -> 13.5 mm
- net Net-(J5-Pad5): track 6.45 -> 4.07 mm
- net Net-(D1-Pad1): track 17.4 -> 19.5 mm
- net Net-(D1-Pad2): track 20.2 -> 22.0 mm
- net Net-(R10-Pad2): track 15.0 -> 16.6 mm
- net Net-(R4-Pad1): track 29.0 -> 30.4 mm
- net Net-(J4-Pad5): track 5.25 -> 5.93 mm
